File: esp-multi-program.sch (KiCad schematic (older format))
At the start: 12 parts, among them P1 CONN_01X08, P2 CONN_01X08, P3 CONN_01X06, P4 CONN_01X02, SW1 PTS645, SW2 PTS645, U1 ESP-12E, U2 ESP-01v090

Commit message: Fixing resistors and adding headers
Parts:
- removed R3: R, Resistors_SMD:R_0805_HandSoldering, symbol R
- added P5: CONN_01X01, Pin_Headers:Pin_Header_Straight_1x01, symbol CONN_01X01
- added R4: 220, Resistors_SMD:R_0805_HandSoldering, symbol R
- R1, R2: value R -> 2.2K
Connections:
- net GPIO_2: now also R4.1; no longer LED1.4 (DIN)
- net at LED1.2 (DOUT): now also P5.1 (P1)
- new net: LED1.4 (DIN), R4.2
Other:
- moved on the sheet: SW2
Changed lines of the file:
@@
 CH_PD
 $Comp
-L GND #PWR01
+L GND #PWR2
 U 1 1 57DD9FA1
 P 1600 4350
-F 0 "#PWR01" H 1600 4100 50  0001 C CNN
+F 0 "#PWR2" H 1600 4100 50  0001 C CNN
 F 1 "GND" H 1600 4200 50  0000 C CNN
 F 2 "" H 1600 4350 50  0000 C CNN
@@
 $EndComp
 $Comp
-L +3.3V #PWR02
+L +3.3V #PWR1
 U 1 1 57DD9FBB
 P 1600 3750
-F 0 "#PWR02" H 1600 3600 50  0001 C CNN
+F 0 "#PWR1" H 1600 3600 50  0001 C CNN
 F 1 "+3.3V" H 1600 3890 50  0000 C CNN
 F 2 "" H 1600 3750 50  0000 C CNN
@@
 $EndComp
 $Comp
-L +3.3V #PWR03
+L +3.3V #PWR3
 U 1 1 57DD9FD9
 P 2450 3750
-F 0 "#PWR03" H 2450 3600 50  0001 C CNN
+F 0 "#PWR3" H 2450 3600 50  0001 C CNN
 F 1 "+3.3V" H 2450 3890 50  0000 C CNN
 F 2 "" H 2450 3750 50  0000 C CNN
@@
 P 2450 4000
 F 0 "R1" V 2530 4000 50  0000 C CNN
-F 1 "R" V 2450 4000 50  0000 C CNN
+F 1 "2.2K" V 2450 4000 50  0000 C CNN
 F 2 "Resistors_SMD:R_0805_HandSoldering" V 2380 4000 50  0001 C CNN
 F 3 "" H 2450 4000 50  0000 C CNN
@@
 VCC
 $Comp
-L PWR_FLAG #FLG04
+L PWR_FLAG #FLG1
 U 1 1 57DDA146
 P 1750 3800
-F 0 "#FLG04" H 1750 3895 50  0001 C CNN
+F 0 "#FLG1" H 1750 3895 50  0001 C CNN
 F 1 "PWR_FLAG" H 1750 3980 50  0000 C CNN
 F 2 "" H 1750 3800 50  0000 C CNN
@@
 GND
 $Comp
-L PWR_FLAG #FLG05
+L PWR_FLAG #FLG2
 U 1 1 57DDA186
 P 1750 4300
-F 0 "#FLG05" H 1750 4395 50  0001 C CNN
+F 0 "#FLG2" H 1750 4395 50  0001 C CNN
 F 1 "PWR_FLAG" H 1750 4480 50  0000 C CNN
 F 2 "" H 1750 4300 50  0000 C CNN
@@
 P 2800 4000
 F 0 "R2" V 2880 4000 50  0000 C CNN
-F 1 "R" V 2800 4000 50  0000 C CNN
+F 1 "2.2K" V 2800 4000 50  0000 C CNN
 F 2 "Resistors_SMD:R_0805_HandSoldering" V 2730 4000 50  0001 C CNN
 F 3 "" H 2800 4000 50  0000 C CNN
@@
 $EndComp
 $Comp
-L +3.3V #PWR06
+L +3.3V #PWR4
 U 1 1 57DDA34E
 P 2800 3750
-F 0 "#PWR06" H 2800 3600 50  0001 C CNN
+F 0 "#PWR4" H 2800 3600 50  0001 C CNN
 F 1 "+3.3V" H 2800 3890 50  0000 C CNN
 F 2 "" H 2800 3750 50  0000 C CNN
@@
 ADC
 $Comp
-L GND #PWR07
+L GND #PWR5
 U 1 1 57DDA662
 P 2800 4700
-F 0 "#PWR07" H 2800 4450 50  0001 C CNN
+F 0 "#PWR5" H 2800 4450 50  0001 C CNN
 F 1 "GND" H 2800 4550 50  0000 C CNN
 F 2 "" H 2800 4700 50  0000 C CNN
@@
 VCC
 $Comp
-L R R3
-U 1 1 57DDADFF
-P 3450 4000
-F 0 "R3" V 3530 4000 50  0000 C CNN
-F 1 "R" V 3450 4000 50  0000 C CNN
-F 2 "Resistors_SMD:R_0805_HandSoldering" V 3380 4000 50  0001 C CNN
-F 3 "" H 3450 4000 50  0000 C CNN
-	1    3450 4000
-	1    0    0    -1
-$EndComp
-$Comp
-L GND #PWR08
+L GND #PWR6
 U 1 1 57DDAE45
-P 3450 4700
-F 0 "#PWR08" H 3450 4450 50  0001 C CNN
-F 1 "GND" H 3450 4550 50  0000 C CNN
-F 2 "" H 3450 4700 50  0000 C CNN
-F 3 "" H 3450 4700 50  0000 C CNN
-	1    3450 4700
-	1    0    0    -1
-$EndComp
-$Comp
-L +3.3V #PWR09
-U 1 1 57DDAE71
-P 3450 3750
-F 0 "#PWR09" H 3450 3600 50  0001 C CNN
-F 1 "+3.3V" H 3450 3890 50  0000 C CNN
-F 2 "" H 3450 3750 50  0000 C CNN
-F 3 "" H 3450 3750 50  0000 C CNN
-	1    3450 3750
-	1    0    0    -1
-$EndComp
-Wire Wire Line
-	3450 4150 3450 4300
-Wire Wire Line
-	3450 3850 3450 3750
-Text Label 3550 4200 0    60   ~ 0
+P 3450 4400
+F 0 "#PWR6" H 3450 4150 50  0001 C CNN
+F 1 "GND" H 3450 4250 50  0000 C CNN
+F 2 "" H 3450 4400 50  0000 C CNN
+F 3 "" H 3450 4400 50  0000 C CNN
+	1    3450 4400
+	1    0    0    -1
+$EndComp
+Text Label 3450 3900 1    60   ~ 0
 GPIO_0
-Wire Wire Line
-	3550 4200 3450 4200
-Connection ~ 3450 4200
 Wire Wire Line
 	2800 4200 2900 4200
@@
 L PTS645 SW2
 U 1 1 57DDBB97
-P 3500 4450
-F 0 "SW2" H 3500 4350 60  0000 C CNN
-F 1 "PTS645" H 3500 4550 60  0000 C CNN
-F 2 "particle:PTS645" H 3500 4450 60  0001 C CNN
-F 3 "" H 3500 4450 60  0001 C CNN
-	1    3500 4450
-	0    1    1    0
-$EndComp
-Wire Wire Line
-	3450 4300 3500 4300
+P 3500 4150
+F 0 "SW2" H 3500 4050 60  0000 C CNN
+F 1 "PTS645" H 3500 4250 60  0000 C CNN
+F 2 "particle:PTS645" H 3500 4150 60  0001 C CNN
+F 3 "" H 3500 4150 60  0001 C CNN
+	1    3500 4150
+	0    1    1    0
+$EndComp
+Wire Wire Line
+	3450 4000 3500 4000
 Wire Wire Line
 	2800 4300 2850 4300
@@
 	2800 4600 2800 4700
 Wire Wire Line
-	3500 4600 3450 4600
-Wire Wire Line
-	3450 4600 3450 4700
+	3500 4300 3450 4300
+Wire Wire Line
+	3450 4300 3450 4400
 $Comp
 L CONN_01X06 P3
@@
 Text Label 2100 5750 0    60   ~ 0
 GND
-Text Label 2100 5350 0    60   ~ 0
+Text Label 2450 5350 0    60   ~ 0
 GPIO_2
+$Comp
+L R R4
+U 1 1 57DDD5C5
+P 2300 5350
+F 0 "R4" V 2380 5350 50  0000 C CNN
+F 1 "220" V 2300 5350 50  0000 C CNN
+F 2 "Resistors_SMD:R_0805_HandSoldering" V 2230 5350 50  0001 C CNN
+F 3 "" H 2300 5350 50  0000 C CNN
+	1    2300 5350
+	0    1    1    0
+$EndComp
+Wire Wire Line
+	2100 5350 2150 5350
+Wire Wire Line
+	3450 3900 3450 4000
+$Comp
+L CONN_01X01 P5
+U 1 1 57DDDD90
+P 900 5750
+F 0 "P5" H 900 5850 50  0000 C CNN
+F 1 "CONN_01X01" V 1000 5750 50  0000 C CNN
+F 2 "Pin_Headers:Pin_Header_Straight_1x01" H 900 5750 50  0001 C CNN
+F 3 "" H 900 5750 50  0000 C CNN
+	1    900  5750
+	-1   0    0    1
+$EndComp
 $EndSCHEMATC
